File: Señal de salida.kicad_sch (KiCad schematic)
At the start: 10 parts, among them J1 Screw_Terminal_01x02, U4 AD9833_Module, U5 X9C103S_Module, U6 TL071

Commit message: Update schematics: signal conditioning, power, ESP32-S3, output, and add signal measurement sub-sheet
Parts:
- C6: footprint (none) -> Capacitor_THT:C_Disc_D7.5mm_W2.5mm_P5.00mm
- J1: footprint (none) -> TerminalBlock:TerminalBlock_MaiXu_MX126-5.0-02P_1x02_P5.00mm
- R2, R4: footprint (none) -> Resistor_THT:R_Axial_DIN0207_L6.3mm_D2.5mm_P10.16mm_Horizontal
- R3: value R -> 50; footprint (none) -> Resistor_THT:R_Axial_DIN0207_L6.3mm_D2.5mm_P10.16mm_Horizontal
- TP2, TP3: footprint (none) -> TestPoint:TestPoint_Loop_D2.50mm_Drill1.0mm
- U6: footprint (none) -> Package_DIP:CERDIP-8_W7.62mm_SideBrazed_LongPads_Socket
Connections:
- net at R2.1, U5.7 (VW): now also U5.6 (VL)
- net GPIO5/ADC1_CH4: now reaches U5.2 (CS)
- net GPIO7/ADC1_CH6: now reaches U5.3 (INC)
- net GPIO6/ADC1_CH5: now reaches U5.4 (U/D)
- no-connect marks 4 -> 3
Changed lines of the file:
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@@
+	)
+	(junction
+		(at 111.76 68.58)
+		(diameter 0)
+		(color 0 0 0 0)
 	)
 	(junction
@@
 	)
 	(no_connect
-		(at 107.95 68.58)
-	)
-	(no_connect
 		(at 168.91 93.98)
 	)
@@
 	(wire
 		(pts
-			(xy 128.27 71.12) (xy 128.27 99.06)
-		)
-		(stroke
-			(width 0)
-			(type default)
-		)
-	)
-	(wire
-		(pts
 			(xy 153.67 83.82) (xy 153.67 99.06)
 		)
@@
 	(wire
 		(pts
+			(xy 128.27 68.58) (xy 128.27 99.06)
+		)
+		(stroke
+			(width 0)
+			(type default)
+		)
+	)
+	(wire
+		(pts
 			(xy 200.66 93.98) (xy 201.93 93.98)
 		)
@@
 	(wire
 		(pts
+			(xy 107.95 68.58) (xy 111.76 68.58)
+		)
+		(stroke
+			(width 0)
+			(type default)
+		)
+	)
+	(wire
+		(pts
 			(xy 163.83 111.76) (xy 163.83 109.22)
 		)
@@
 	(wire
 		(pts
-			(xy 107.95 71.12) (xy 128.27 71.12)
+			(xy 107.95 71.12) (xy 111.76 71.12)
 		)
 		(stroke
@@
 	(wire
 		(pts
+			(xy 111.76 71.12) (xy 111.76 68.58)
+		)
+		(stroke
+			(width 0)
+			(type default)
+		)
+	)
+	(wire
+		(pts
 			(xy 107.95 99.06) (xy 111.76 99.06)
 		)
@@
 		(pts
 			(xy 82.55 96.52) (xy 80.01 96.52)
+		)
+		(stroke
+			(width 0)
+			(type default)
+		)
+	)
+	(wire
+		(pts
+			(xy 111.76 68.58) (xy 128.27 68.58)
 		)
 		(stroke
@@
 		)
 	)
+	(hierarchical_label "GPIO7/ADC1_CH6"
+		(shape bidirectional)
+		(at 82.55 71.12 180)
+		(effects
+			(font
+				(size 1.27 1.27)
+			)
+			(justify right)
+		)
+	)
 	(hierarchical_label "V-"
 		(shape input)
@@
 		)
 	)
+	(hierarchical_label "GPIO5/ADC1_CH4"
+		(shape bidirectional)
+		(at 82.55 68.58 180)
+		(effects
+			(font
+				(size 1.27 1.27)
+			)
+			(justify right)
+		)
+	)
 	(hierarchical_label "5V"
 		(shape input)
 		(at 76.2 66.04 180)
+		(effects
+			(font
+				(size 1.27 1.27)
+			)
+			(justify right)
+		)
+	)
+	(hierarchical_label "GPIO6/ADC1_CH5"
+		(shape bidirectional)
+		(at 82.55 73.66 180)
 		(effects
 			(font
@@
 			)
 		)
-		(property "Footprint" ""
+		(property "Footprint" "TestPoint:TestPoint_Loop_D2.50mm_Drill1.0mm"
 			(at 205.74 90.17 0)
 			(hide yes)
@@
 			)
 		)
-		(property "Footprint" ""
+		(property "Footprint" "Resistor_THT:R_Axial_DIN0207_L6.3mm_D2.5mm_P10.16mm_Horizontal"
 			(at 166.37 85.598 90)
 			(hide yes)
@@
 			)
 		)
-		(property "Footprint" ""
+		(property "Footprint" "Resistor_THT:R_Axial_DIN0207_L6.3mm_D2.5mm_P10.16mm_Horizontal"
 			(at 140.97 100.838 90)
 			(hide yes)
@@
 			)
 		)
-		(property "Value" "R"
+		(property "Value" "50"
 			(at 189.23 97.79 90)
 			(show_name no)
@@
 			)
 		)
-		(property "Footprint" ""
+		(property "Footprint" "Resistor_THT:R_Axial_DIN0207_L6.3mm_D2.5mm_P10.16mm_Horizontal"
 			(at 189.23 103.378 90)
 			(hide yes)
@@
 			)
 		)
-		(property "Footprint" ""
+		(property "Footprint" "TerminalBlock:TerminalBlock_MaiXu_MX126-5.0-02P_1x02_P5.00mm"
 			(at 214.63 101.6 0)
 			(hide yes)
@@
 			)
 		)
-		(property "Footprint" ""
+		(property "Footprint" "Package_DIP:CERDIP-8_W7.62mm_SideBrazed_LongPads_Socket"
 			(at 167.64 102.87 0)
 			(hide yes)
@@
 			)
 		)
-		(property "Footprint" ""
+		(property "Footprint" "Capacitor_THT:C_Disc_D7.5mm_W2.5mm_P5.00mm"
 			(at 119.38 98.0948 0)
 			(hide yes)
@@
 			)
 		)
-		(property "Footprint" ""
+		(property "Footprint" "TestPoint:TestPoint_Loop_D2.50mm_Drill1.0mm"
 			(at 128.27 62.23 0)
 			(hide yes)
