File: TD3-FrequencyAnalizer.kicad_pcb (KiCad board)
At the start: 0 parts

Commit message: Update project files and add schematic sheets (ESP32-S3, Alimentacion, Acondicionamiento, Salida)
Parts:
- added U1: ESP32-S3-DevKitC, Espressif:ESP32-S3-DevKitC, F.Cu at (96.7, 55.6)
Other:
- copper layers 0 -> 2

Commit message: Save local schematic and board updates before 3D model path resolution
Parts:
- added C1: 1uF, Capacitor_THT:C_Disc_D7.5mm_W2.5mm_P5.00mm, F.Cu at (40.8, 271.0)
- added C10: C, Capacitor_THT:C_Disc_D7.5mm_W2.5mm_P5.00mm, F.Cu at (329.5, 71.7)
- added C11: 1uF, Capacitor_THT:C_Disc_D7.5mm_W2.5mm_P5.00mm, F.Cu at (329.5, 75.7)
- added C12: C, Capacitor_THT:C_Disc_D7.5mm_W2.5mm_P5.00mm, F.Cu at (329.5, 79.8)
- added C13: C, Capacitor_THT:C_Disc_D7.5mm_W2.5mm_P5.00mm, F.Cu at (329.5, 83.8)
- added C14: C, Capacitor_THT:C_Disc_D7.5mm_W2.5mm_P5.00mm, F.Cu at (329.5, 87.9)
- added C2: 100nF, Capacitor_THT:C_Disc_D7.5mm_W2.5mm_P5.00mm, F.Cu at (-161.9, -224.6)
- added C3: 100nF, Capacitor_THT:C_Disc_D7.5mm_W2.5mm_P5.00mm, F.Cu at (-161.9, -220.6)
- added C4: 100nF, Capacitor_THT:C_Disc_D7.5mm_W2.5mm_P5.00mm, F.Cu at (-161.9, -216.5)
- added C5: 100nF, Capacitor_THT:C_Disc_D7.5mm_W2.5mm_P5.00mm, F.Cu at (-161.9, -212.5)
- added C6: 1uF, Capacitor_THT:C_Disc_D7.5mm_W2.5mm_P5.00mm, F.Cu at (100.7, 60.9)
- added C7: 100nF, Capacitor_THT:C_Disc_D7.5mm_W2.5mm_P5.00mm, F.Cu at (52.1, 66.7)
- added C8: 100nF, Capacitor_THT:C_Disc_D7.5mm_W2.5mm_P5.00mm, F.Cu at (61.9, 73.4)
- added D2: BAT54S, Package_TO_SOT_SMD:SOT-23, B.Cu at (422.1, 59.3)
- added D3: 1N4001, Diode_THT:D_DO-41_SOD81_P10.16mm_Horizontal, F.Cu at (328.0, -37.4)
- added D4: BAT54S, Package_TO_SOT_SMD:SOT-23, B.Cu at (95.1, 256.3)
- added J1: Screw_Terminal_01x02, TerminalBlock:TerminalBlock_MaiXu_MX126-5.0-02P_1x02_P5.00mm, F.Cu at (41.6, 62.7)
- added J2: Screw_Terminal_01x03, TerminalBlock:TerminalBlock_MaiXu_MX126-5.0-03P_1x03_P5.00mm, F.Cu at (-155.0, -174.7)
- added J3: Screw_Terminal_01x02, TerminalBlock:TerminalBlock_MaiXu_MX126-5.0-02P_1x02_P5.00mm, F.Cu at (-147.5, -159.4)
- added K1: G6A, Relay_THT:Relay_DPDT_Omron_G6A, F.Cu at (328.3, 42.8)
- added Q1: BC547, Package_TO_SOT_THT:TO-92_HandSolder, F.Cu at (394.2, 10.5)
- added R10: R, Resistor_THT:R_Axial_DIN0207_L6.3mm_D2.5mm_P10.16mm_Horizontal, F.Cu at (327.7, -13.0)
- added R11: R, Resistor_THT:R_Axial_DIN0207_L6.3mm_D2.5mm_P10.16mm_Horizontal, F.Cu at (327.7, -9.00)
- added R12: R, Resistor_THT:R_Axial_DIN0207_L6.3mm_D2.5mm_P10.16mm_Horizontal, F.Cu at (327.7, -4.95)
- added R13: 1M, Resistor_THT:R_Axial_DIN0207_L6.3mm_D2.5mm_P10.16mm_Horizontal, F.Cu at (327.7, -0.90)
- added R14: R, Resistor_THT:R_Axial_DIN0207_L6.3mm_D2.5mm_P10.16mm_Horizontal, F.Cu at (327.7, 3.15)
- added R15: R, Resistor_THT:R_Axial_DIN0207_L6.3mm_D2.5mm_P10.16mm_Horizontal, F.Cu at (327.7, 7.20)
- added R16: R, Resistor_THT:R_Axial_DIN0207_L6.3mm_D2.5mm_P10.16mm_Horizontal, F.Cu at (327.7, 11.3)
- added R17: R, Resistor_THT:R_Axial_DIN0207_L6.3mm_D2.5mm_P10.16mm_Horizontal, F.Cu at (327.7, 15.3)
- added R18: R, Resistor_THT:R_Axial_DIN0207_L6.3mm_D2.5mm_P10.16mm_Horizontal, F.Cu at (327.7, 19.4)
- added R19: R, Resistor_THT:R_Axial_DIN0207_L6.3mm_D2.5mm_P10.16mm_Horizontal, F.Cu at (27.0, 249.6)
- added R2: R, Resistor_THT:R_Axial_DIN0207_L6.3mm_D2.5mm_P10.16mm_Horizontal, F.Cu at (84.1, 73.3)
- added R20: R, Resistor_THT:R_Axial_DIN0207_L6.3mm_D2.5mm_P10.16mm_Horizontal, F.Cu at (327.7, 23.4)
- added R21: R, Resistor_THT:R_Axial_DIN0207_L6.3mm_D2.5mm_P10.16mm_Horizontal, F.Cu at (-153.3, -224.6)
- added R22: R, Resistor_THT:R_Axial_DIN0207_L6.3mm_D2.5mm_P10.16mm_Horizontal, F.Cu at (-153.3, -220.6)
- added R23: R, Resistor_THT:R_Axial_DIN0207_L6.3mm_D2.5mm_P10.16mm_Horizontal, F.Cu at (-153.3, -216.5)
- added R24: R, Resistor_THT:R_Axial_DIN0207_L6.3mm_D2.5mm_P10.16mm_Horizontal, F.Cu at (-153.3, -212.5)
- added R25: R, Resistor_THT:R_Axial_DIN0207_L6.3mm_D2.5mm_P10.16mm_Horizontal, F.Cu at (327.7, 27.5)
- added R26: R, Resistor_THT:R_Axial_DIN0207_L6.3mm_D2.5mm_P10.16mm_Horizontal, F.Cu at (327.7, 31.5)
- added R27: R, Resistor_THT:R_Axial_DIN0207_L6.3mm_D2.5mm_P10.16mm_Horizontal, F.Cu at (27.0, 253.6)
- added R28: R, Resistor_THT:R_Axial_DIN0207_L6.3mm_D2.5mm_P10.16mm_Horizontal, F.Cu at (27.0, 257.7)
- added R29: R, Resistor_THT:R_Axial_DIN0207_L6.3mm_D2.5mm_P10.16mm_Horizontal, F.Cu at (27.0, 261.7)
- added R3: 50, Resistor_THT:R_Axial_DIN0207_L6.3mm_D2.5mm_P10.16mm_Horizontal, F.Cu at (74.0, 69.1)
- added R31: R, Resistor_THT:R_Axial_DIN0207_L6.3mm_D2.5mm_P10.16mm_Horizontal, F.Cu at (27.0, 265.8)
- added R33: R, Resistor_THT:R_Axial_DIN0207_L6.3mm_D2.5mm_P10.16mm_Horizontal, F.Cu at (27.0, 269.8)
- added R34: R, Resistor_THT:R_Axial_DIN0207_L6.3mm_D2.5mm_P10.16mm_Horizontal, F.Cu at (27.0, 273.9)
- added R4: R, Resistor_THT:R_Axial_DIN0207_L6.3mm_D2.5mm_P10.16mm_Horizontal, F.Cu at (84.1, 64.2)
- added R5: R, Resistor_THT:R_Axial_DIN0207_L6.3mm_D2.5mm_P10.16mm_Horizontal, F.Cu at (327.7, -33.3)
- added R6: R, Resistor_THT:R_Axial_DIN0207_L6.3mm_D2.5mm_P10.16mm_Horizontal, F.Cu at (327.7, -29.2)
- added R7: R, Resistor_THT:R_Axial_DIN0207_L6.3mm_D2.5mm_P10.16mm_Horizontal, F.Cu at (327.7, -25.2)
- added R8: R, Resistor_THT:R_Axial_DIN0207_L6.3mm_D2.5mm_P10.16mm_Horizontal, F.Cu at (327.7, -21.1)
- added R9: R, Resistor_THT:R_Axial_DIN0207_L6.3mm_D2.5mm_P10.16mm_Horizontal, F.Cu at (327.7, -17.1)
- added RV2: R_Potentiometer_Trim, Potentiometer_THT:Potentiometer_Bourns_3266Y_Vertical, F.Cu at (347.3, 19.6)
- added RV3: R_Potentiometer_Trim, Potentiometer_THT:Potentiometer_Bourns_3266Y_Vertical, F.Cu at (-157.2, -199.4)
- added RV4: R_Potentiometer_Trim, Potentiometer_THT:Potentiometer_Bourns_3266Y_Vertical, F.Cu at (-157.2, -193.3)
- added RV5: R_Potentiometer_Trim, Potentiometer_THT:Potentiometer_Bourns_3266Y_Vertical, F.Cu at (45.4, 250.5)
- added RV6: R_Potentiometer_Trim, Potentiometer_THT:Potentiometer_Bourns_3266Y_Vertical, F.Cu at (347.3, 25.6)
- added RV7: R_Potentiometer_Trim, Potentiometer_THT:Potentiometer_Bourns_3266Y_Vertical, F.Cu at (45.4, 256.6)
- added TP2: Señal de Salida, TestPoint:TestPoint_Loop_D2.50mm_Drill1.0mm, F.Cu at (73.7, 92.8)
- added TP3: Señal AD9833, TestPoint:TestPoint_Loop_D2.50mm_Drill1.0mm, F.Cu at (73.7, 97.5)
- added TP4: TestPoint, TestPoint:TestPoint_Loop_D2.50mm_Drill1.0mm, F.Cu at (402.1, -2.04)
- added TP5: TestPoint, TestPoint:TestPoint_Loop_D2.50mm_Drill1.0mm, F.Cu at (402.1, 2.61)
- added TP6: TestPoint, TestPoint:TestPoint_Loop_D2.50mm_Drill1.0mm, F.Cu at (41.1, 262.0)
- added TP7: TestPoint, TestPoint:TestPoint_Loop_D2.50mm_Drill1.0mm, F.Cu at (41.1, 266.6)
- added U2: TL074, Package_DIP:CERDIP-14_W7.62mm_SideBrazed_LongPads_Socket, F.Cu at (406.2, -29.3)
- added U3: TL072, Package_DIP:CERDIP-8_W7.62mm_SideBrazed_LongPads_Socket, F.Cu at (-143.7, -192.3)
- added U4: AD9833_Module, AD9833_Module:AD9833_Module, F.Cu at (111.7, 89.7)
- added U5: X9C103S_Module, X9C103S_Module:X9C103S_Module, F.Cu at (100.2, 70.7)
- added U6: TL071, Package_DIP:CERDIP-8_W7.62mm_SideBrazed_LongPads_Socket, F.Cu at (58.3, 68.0)
- moved U1 27.5 mm to (121.9, 44.9)
Connections:
- net Net-(U1-GND-Pad22) renamed GND
- U1 pad 1: Net-(U1-3V3-Pad1) -> unconnected-(U1-3V3-Pad1)
- U1 pad 16: unconnected-(U1-GPIO10/ADC1_CH9-Pad16) -> /ESP32-S3/GPIO10/ADC1_CH9
- U1 pad 17: unconnected-(U1-GPIO11/ADC2_CH0-Pad17) -> /ESP32-S3/GPIO11/ADC2_CH0
- U1 pad 18: unconnected-(U1-GPIO12/ADC2_CH1-Pad18) -> /ESP32-S3/GPIO12/ADC2_CH1
- U1 pad 2: Net-(U1-3V3-Pad1) -> unconnected-(U1-3V3-Pad1)_1
- U1 pad 21: unconnected-(U1-5V-Pad21) -> /ESP32-S3/5V
- U1 pad 4: unconnected-(U1-GPIO4/ADC1_CH3-Pad4) -> /Acondicionamiento de Señal de Entrada/GPIO4/ADC1_CH3
- U1 pad 40: unconnected-(U1-GPIO2/ADC1_CH1-Pad40) -> /Acondicionamiento de Señal de Entrada/GPIO2/ADC1_CH1
- U1 pad 41: unconnected-(U1-GPIO1/ADC1_CH0-Pad41) -> /ESP32-S3/GPIO1/ADC1_CH0
- U1 pad 5: unconnected-(U1-GPIO5/ADC1_CH4-Pad5) -> /ESP32-S3/GPIO5/ADC1_CH4
- U1 pad 6: unconnected-(U1-GPIO6/ADC1_CH5-Pad6) -> /ESP32-S3/GPIO6/ADC1_CH5
- U1 pad 7: unconnected-(U1-GPIO7/ADC1_CH6-Pad7) -> /ESP32-S3/GPIO7/ADC1_CH6
Routing:
- net /ESP32-S3/5V: track 0.00 -> 32.2 mm
- net /ESP32-S3/GPIO5/ADC1_CH4: track 0.00 -> 30.5 mm
- net /ESP32-S3/GPIO11/ADC2_CH0: track 0.00 -> 22.0 mm
- net /ESP32-S3/GPIO7/ADC1_CH6: track 0.00 -> 21.5 mm
- net /ESP32-S3/GPIO6/ADC1_CH5: track 0.00 -> 20.5 mm
- net Net-(R3-Pad1): track 0.00 -> 18.4 mm
- net Net-(U6--): track 0.00 -> 17.7 mm
- net +12V: track 0.00 -> 11.8 mm
- net /ESP32-S3/GPIO10/ADC1_CH9: track 0.00 -> 10.9 mm
- net Net-(U5-VH): track 0.00 -> 10.8 mm
- net /ESP32-S3/GPIO12/ADC2_CH1: track 0.00 -> 10.6 mm
- net Net-(U5-VL): track 0.00 -> 7.21 mm
- net -12V: track 0.00 -> 5.81 mm
Other:
- board outline added: 179.3 x 113.2 mm

Commit message: Update PCB layout: Component placements, routing and 3D model alignments
Parts:
- moved C4 484.0 mm to (187.5, 118.5), turned to -90 degrees
- moved C5 467.8 mm to (163.7, 123.5), turned to 90 degrees
- moved J3 442.7 mm to (207.9, 104.7), turned to -90 degrees
- moved C2 436.6 mm to (171.7, 57.2), turned to 90 degrees
- moved C3 415.8 mm to (156.0, 47.4)
- moved U3 393.2 mm to (165.3, 50.9), turned to -90 degrees
- moved R34 278.1 mm to (175.8, 38.9), turned to -90 degrees
- moved R33 276.9 mm to (179.7, 38.9), turned to -90 degrees
- moved U2 266.8 mm to (183.2, 117.2), turned to -90 degrees
- moved R31 265.5 mm to (165.9, 39.5), turned to 180 degrees
- moved C1 260.8 mm to (169.1, 43.9), turned to 90 degrees
- moved Q1 260.6 mm to (152.5, 107.8), turned to 90 degrees
- moved RV7 252.6 mm to (185.8, 46.5), turned to -90 degrees
- moved TP4 251.0 mm to (187.9, 128.9)
- moved TP5 245.1 mm to (199.1, 140.1)
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Routing:
- net /Medición de Señal Inyectada/OutputSignal: track 0.00 -> 140.1 mm
- net /ESP32-S3/GPIO1/ADC1_CH0: track 0.00 -> 54.6 mm
- net Net-(U2B--): track 0.00 -> 53.8 mm
- net Net-(R27-Pad1): track 0.00 -> 52.1 mm
- net Net-(U3B--): track 0.00 -> 50.0 mm
- net Net-(U2B-+): track 0.00 -> 44.1 mm
- net /Acondicionamiento de Señal de Entrada/K1_21: track 0.00 -> 34.9 mm
- net Net-(C1-Pad2): track 0.00 -> 30.4 mm
- net +12V: track 11.8 -> 41.6 mm
- net /Acondicionamiento de Señal de Entrada/K1_11: track 0.00 -> 26.4 mm
- net Net-(U2C-+): track 0.00 -> 20.8 mm
- net /Acondicionamiento de Señal de Entrada/K1_A2: track 0.00 -> 20.5 mm
- net -12V: track 5.81 -> 24.9 mm
- net Net-(U3A--): track 0.00 -> 17.5 mm
- net Net-(U2D--): track 0.00 -> 16.1 mm
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- added copper zone on B.Cu, net GND
